Commit message: SLAM enabled, manual PID needs work
Hardware interface adapted, not tested. Description file finished. All dependencies added to CMakeLists. Lidar transform to base_link working. EKF implemented for wheel odometry and lidar odometry, tested with ros2_laser_scan_matcher. Slam toolbox tested and working with mapper..yaml parameters.

File: ros2/robotic_description/urdf/robotic.urdf.xacro (robot description, xacro)
@@ -1,22 +1,18 @@
 <?xml version="1.0"?>
 <robot name="robotic" xmlns:xacro="http://ros.org/wiki/xacro">
-  <xacro:include filename="ros2_control.xacro" />
+  <!-- <xacro:include filename="$(find robotic_description)/urdf/robotic.gazebo" /> -->
   <!-- ****************** ROBOT CONSTANTS *******************************  -->
-  <!-- Define the size of the robot's main chassis in meters -->
-  <xacro:property name="base_width"
-    value="0.160" />
+  <!-- Define the siz.e of the robot's main chassis in meters -->
+  <xacro:property name="base_width" value="0.160" />
   <xacro:property name="base_length" value="0.120" />
-  <xacro:property
-    name="base_height" value="0.160" />
+  <xacro:property name="base_height" value="0.160" />
   <!-- Define the shape of the robot's two back wheels in meters -->
-  <xacro:property name="wheel_radius" value="${0.072/2}" />
-  <xacro:property
-    name="wheel_width" value="0.0124" />
+  <xacro:property name="wheel_radius" value="0.035" />
+  <xacro:property name="wheel_width" value="0.0124" />
   <!-- x-axis points forward, y-axis points to left, z-axis points upwards -->
   <!-- Define the gap between the wheel and chassis along y-axis in meters -->
   <xacro:property name="wheel_ygap" value="0.0" /> , <!--
   Position the wheels along the z-axis -->
-  <xacro:property
-    name="wheel_zoff" value="${0.012+wheel_radius}" />
+  <xacro:property name="wheel_zoff" value="${0.012+wheel_radius}" />
   <!-- Position the wheels along the x-axis -->
   <xacro:property name="wheel_xoff" value="0.0" />
@@ -52,7 +48,7 @@
   <!-- The base footprint of the robot is located underneath the chassis -->
   <joint
-    name="base_joint" type="fixed">
-    <parent link="base_footprint" />
-    <child link="base_link" />
+    name="base_footprint_joint" type="fixed">
+    <parent link="base_link" />
+    <child link="base_footprint" />
     <origin xyz="0.0 0.0 ${(wheel_radius+wheel_zoff)}" rpy="0 0 0" />
   </joint>
@@ -74,5 +70,5 @@
       </geometry>
     </collision>
-    <xacro:box_inertia m="40.0" w="${base_width}" d="${base_length}" h="${base_height}" />
+    <!-- <xacro:box_inertia m="40.0" w="${base_width}" d="${base_length}" h="${base_height}" /> -->
   </link>
   <gazebo
@@ -92,5 +88,5 @@
         </material>
       </visual>
-      <collision>
+      <collision>180
         <origin xyz="0 0 0" rpy="${pi/2} 0 0" />
         <geometry>
@@ -98,15 +94,15 @@
         </geometry>
       </collision>
-      <xacro:cylinder_inertia m="0.5" r="${wheel_radius}" h="${wheel_width}" />
+      <xacro:cylinder_inertia m="0.1" r="${wheel_radius}" h="${wheel_width}" />
     </link>
     <!-- Connect the wheels to the base_link at the appropriate location, and
          define a continuous joint to allow the wheels to freely rotate about
          an axis -->
-    <joint name="${prefix}_joint" type="revolute">
+    <joint name="${prefix}_joint" type="continuous">
       <parent link="base_link" />
       <child link="${prefix}_link" />
       <origin xyz="${x_reflect*wheel_xoff} ${y_reflect*(base_width/2+wheel_ygap)} ${-wheel_zoff}"
         rpy="0 0 0" />
-      <limit upper="3.1415" lower="-3.1415" effort="30" velocity="5.0" />
+      <!-- <limit upper="3.1415" lower="-3.1415" effort="30" velocity="5.0" /> -->
       <axis xyz="0 1 0" />
     </joint>
@@ -117,5 +113,5 @@
   <xacro:wheel prefix="left_wheel" x_reflect="0" y_reflect="1" />
   <xacro:wheel prefix="right_wheel" x_reflect="0" y_reflect="-1" />
-  *********************** TEFLON ******************************
+  <!-- *********************** TEFLON ******************************  -->
   <link name="teflon">
     <visual>
@@ -130,5 +126,5 @@
       <origin xyz="0.0 0.0 0.0" rpy="0.0 0.0 0.0"/>
       <geometry>
-        <box size="0.013 0.46 0.0247"/>
+        <box size="0.013 0.102 0.0247"/>
       </geometry>
     </collision>
@@ -145,5 +141,5 @@
     <parent link="base_link" />
     <child link="camera_link" />
-    <origin xyz="0.075 0 -0.02" rpy="0 ${pi/2} 0" />
+    <origin xyz="-0.085 0 -0.02" rpy="0 ${pi/2} 0" />
   </joint>
   <link name="camera_link">
@@ -160,10 +156,10 @@
   <!-- *********************** LIDAR SETUP **********************************  -->
   <joint
-    name="lidar_joint" type="fixed">
+    name="laser_joint" type="fixed">
     <parent link="base_link" />
-    <child link="lidar_link" />
+    <child link="laser" />
     <origin xyz="0 0 0.07" rpy="0 0 0" />
   </joint>
-  <link name="lidar_link">
+  <link name="laser">
     <collision>
       <origin xyz="0 0 0" rpy="0 0 0" />
@@ -187,77 +183,3 @@
     </inertial>
   </link>
-  <gazebo
-    reference="lidar_link">
-    <sensor name="lidar" type="ray">
-      <always_on>true</always_on>
-      <visualize>true</visualize>
-      <update_rate>5</update_rate>
-      <ray>
-        <scan>
-          <horizontal>
-            <samples>120</samples>
-            <resolution>1.000000</resolution>
-            <min_angle>-3.14159</min_angle>
-            <max_angle>3.14159</max_angle>
-          </horizontal>
-        </scan>
-        <range>
-          <min>0.3</min>
-          <max>15.0</max>
-          <resolution>0.015</resolution>
-        </range>
-        <noise>
-          <type>gaussian</type>
-          <mean>0.0</mean>
-          <stddev>0.01</stddev>
-        </noise>
-      </ray>
-      <plugin name="scan" filename="libgazebo_ros_ray_sensor.so">
-        <ros>
-          <remapping>~/out:=scan</remapping>
-        </ros>
-        <output_type>sensor_msgs/LaserScan</output_type>
-        <frame_name>lidar_link</frame_name>
-      </plugin>
-    </sensor>
-  </gazebo>
-  <gazebo
-    reference="lidar_link">
-    <mu1>0.01</mu1>
-    <mu2>0.01</mu2>
-    <material>Gazebo/Black</material>
-  </gazebo>
-  <!-- *********************** WHEEL ODOMETRY ***************************    -->
-  <gazebo>
-    <plugin name="two_wheeled_robot_diff_drive" filename="libgazebo_ros_diff_drive.so">
-      <update_rate>30</update_rate>
-      <!--wheels -->
-      <left_joint>left_wheel_joint</left_joint>
-      <right_joint>right_wheel_joint</right_joint>
-      <!-- kinematics -->
-      <wheel_separation>0.52</wheel_separation>
-      <wheel_diameter>0.28</wheel_diameter>
-      <!-- limits -->
-      <max_wheel_torque>20</max_wheel_torque>
-      <max_wheel_acceleration>1.0</max_wheel_acceleration>
-      <!-- Receive velocity commands on this ROS topic -->
-      <command_topic>cmd_vel</command_topic>
-      <!-- output -->
-      <!-- When false, publish no wheel odometry data to a ROS topic -->
-      <publish_odom>true</publish_odom>
-      <!-- When true, publish coordinate transform from odom to base_footprint -->
-      <!-- I usually use the robot_localization package to publish this transform -->
-      <publish_odom_tf>false</publish_odom_tf>
-      <!-- When true, publish coordinate transform from base_link to the wheels -->
-      <!-- The robot_state_publisher package is often used to publish this transform -->
-      <publish_wheel_tf>true</publish_wheel_tf>
-      <odometry_topic>odom</odometry_topic>
-      <odometry_frame>odom</odometry_frame>
-      <robot_base_frame>base_link</robot_base_frame>
-      <odometry_source>1</odometry_source>
-      <ros>
-        <remapping>odom:=wheel/odometry</remapping>
-      </ros>
-    </plugin>
-  </gazebo>
 </robot>

Commit message: Movement node PID working, frame transforms working
SLAM workiing very well because laser->base_link transform is finally correct in robot URDF. Movement node manipulation through commands working very well - goal_theta is the final angle after movement. All dependencies defined in CMakeLists.txt and package.xml of robotic_pkg, no more need for sllidar package to be a subdirectory.

File: ros2/robotic_description/urdf/robotic.urdf.xacro (robot description, xacro)
@@ -159,5 +159,5 @@
     <parent link="base_link" />
     <child link="laser" />
-    <origin xyz="0 0 0.07" rpy="0 0 0" />
+    <origin xyz="0 0 0.07" rpy="${pi} 0 ${pi}" />
   </joint>
   <link name="laser">
